File: TestBoards/DRV-Tester/DRV-Tester/DRV-Tester.kicad_pcb (KiCad board)
At the start: 2 copper layers, 0 parts

Commit message: update new tester board sch
Parts:
- added J1: Screw_Terminal_01x02, easyeda2kicad:CONN-TH_P5.08_KF128-5.08-2P, F.Cu at (119.0, 98.7)
- added J10: Conn_02x04_Odd_Even, Connector_PinHeader_2.54mm:PinHeader_2x04_P2.54mm_Vertical, F.Cu at (106.1, 133.5)
- added J11: Conn_02x04_Odd_Even, Connector_PinHeader_2.54mm:PinHeader_2x04_P2.54mm_Vertical, F.Cu at (131.2, 130.6)
- added J2: Screw_Terminal_01x02, easyeda2kicad:CONN-TH_P5.08_KF128-5.08-2P, F.Cu at (92.7, 66.8)
- added J3: Screw_Terminal_01x02, easyeda2kicad:CONN-TH_P5.08_KF128-5.08-2P, F.Cu at (105.4, 99.2)
- added J4: Screw_Terminal_01x02, easyeda2kicad:CONN-TH_P5.08_KF128-5.08-2P, F.Cu at (92.4, 89.5)
- added J5: Screw_Terminal_01x02, easyeda2kicad:CONN-TH_P5.08_KF128-5.08-2P, F.Cu at (135.6, 98.5)
- added J6: Screw_Terminal_01x02, easyeda2kicad:CONN-TH_P5.08_KF128-5.08-2P, F.Cu at (92.4, 78.1)
- added J7: Conn_02x04_Odd_Even, Connector_PinHeader_2.54mm:PinHeader_2x04_P2.54mm_Vertical, F.Cu at (103.7, 116.7)
- added J8: Conn_02x04_Odd_Even, Connector_PinHeader_2.54mm:PinHeader_2x04_P2.54mm_Vertical, F.Cu at (134.0, 117.7)
- added J9: Conn_02x04_Odd_Even, Connector_PinHeader_2.54mm:PinHeader_2x04_P2.54mm_Vertical, F.Cu at (117.6, 117.7)
- added R_IPROP1: 820, Resistor_SMD:R_0603_1608Metric, F.Cu at (196.8, 101.0)
- added R_IPROP2: 820, Resistor_SMD:R_0603_1608Metric, F.Cu at (196.8, 94.0)
- added R_IPROP3: 820, Resistor_SMD:R_0603_1608Metric, F.Cu at (196.8, 87.0)
- added R_nFAULT1: 820, Resistor_SMD:R_0603_1608Metric, F.Cu at (196.8, 89.5)
- added R_nFAULT2: 820, Resistor_SMD:R_0603_1608Metric, F.Cu at (196.8, 96.5)
- added R_nFAULT3: 820, Resistor_SMD:R_0603_1608Metric, F.Cu at (196.8, 103.5)
- added R_nSLEEP1: 8.2k, Resistor_SMD:R_0603_1608Metric, F.Cu at (162.5, 87.2)
- added R_nSLEEP2: 8.2k, Resistor_SMD:R_0603_1608Metric, F.Cu at (150.9, 93.9)
- added R_nSLEEP3: 8.2k, Resistor_SMD:R_0603_1608Metric, F.Cu at (155.8, 121.5)
- added U1: PDRV8244SPWPQ1, PDRV8244SDGQQ1:U_DGQ0028A_TEX-L, F.Cu at (105.3, 109.6)
- added U2: PDRV8245SPWPQ1, PDRV8245SPWPQ1:U_PWP0028R_TEX, F.Cu at (135.3, 109.5)
- added U3: PDRV8243SPWPQ1, PDRV8243SDGQQ:VSSOP_SDGQQ1_TEX, F.Cu at (118.7, 109.6)
- added U4: XT30PW-F, easyeda2kicad:CONN-TH_XT30PW-F-1, F.Cu at (146.0, 109.1)
