File: TestBoards/DRV-Tester/DRV-Tester/DRV8243.kicad_sch (KiCad schematic)
At the start: 0 parts

Commit message: update new tester board sch
Parts:
- added R_IPROP3, R_nFAULT1: 820, Resistor_SMD:R_0603_1608Metric, symbol Device:R_US
- added R_nSLEEP3: 8.2k, Resistor_SMD:R_0603_1608Metric, symbol Device:R_US
- added U3: PDRV8243SPWPQ1, PDRV8243SDGQQ:VSSOP_SDGQQ1_TEX, symbol PDRV8245SPWPQ1:PDRV8245SPWPQ1
Connections:
- new net 3V3_VCC: R_nFAULT1.1
- new net DRV1_CS: U3.2 (NSCS)
- new net DRVOFF: U3.5 (DRVOFF)
- new net GND: R_IPROP3.2, R_nSLEEP3.1, U3.12 (GND), U3.13 (GND), U3.14 (GND), U3.15 (GND), U3.16 (GND), U3.17 (GND), U3.EPAD
- new net IN1: U3.4 (EN/IN1)
- new net IN2: U3.3 (PH/IN2)
- new net IPROPI_1: R_IPROP3.1
- new net IPROPI_2: U3.25 (IPROPI)
- new net M_MISO: U3.27 (SDO)
- new net M_MOSI: U3.28 (SDI)
- new net M_SCLK: U3.1 (SCLK)
- new net NFAULT_1: R_nFAULT1.2, U3.26 (NFAULT)
- new net NSLEEP: R_nSLEEP3.2, U3.24 (NSLEEP)
- new net OUT1: U3.10 (OUT1), U3.11 (OUT1), U3.9 (OUT1)
- new net OUT2: U3.18 (OUT2), U3.19 (OUT2), U3.20 (OUT2)
- new net VM: U3.21 (VM), U3.22 (VM), U3.23 (VM), U3.6 (VM), U3.7 (VM), U3.8 (VM)
