File: TestBoards/DRV-Tester/DRV-Tester/DRV8244.kicad_sch (KiCad schematic)
At the start: 0 parts

Commit message: update new tester board sch
Parts:
- added R_IPROP2, R_nFAULT2: 820, Resistor_SMD:R_0603_1608Metric, symbol Device:R_US
- added R_nSLEEP2: 8.2k, Resistor_SMD:R_0603_1608Metric, symbol Device:R_US
- added U1: PDRV8244SPWPQ1, PDRV8244SDGQQ1:U_DGQ0028A_TEX-L, symbol PDRV8245SPWPQ1:PDRV8245SPWPQ1
Connections:
- new net 3V3_VCC: R_nFAULT2.1
- new net DRV2_CS: U1.2 (NSCS)
- new net DRVOFF: U1.5 (DRVOFF)
- new net GND: R_IPROP2.2, R_nSLEEP2.1, U1.12 (GND), U1.13 (GND), U1.14 (GND), U1.15 (GND), U1.16 (GND), U1.17 (GND), U1.EPAD
- new net IN1: U1.4 (EN/IN1)
- new net IN2: U1.3 (PH/IN2)
- new net IPROPI_2: R_IPROP2.1, U1.25 (IPROPI)
- new net M_MISO: U1.27 (SDO)
- new net M_MOSI: U1.28 (SDI)
- new net M_SCLK: U1.1 (SCLK)
- new net NFAULT_2: R_nFAULT2.2, U1.26 (NFAULT)
- new net NSLEEP: R_nSLEEP2.2, U1.24 (NSLEEP)
- new net OUT1: U1.10 (OUT1), U1.11 (OUT1), U1.9 (OUT1)
- new net OUT2: U1.18 (OUT2), U1.19 (OUT2), U1.20 (OUT2)
- new net VM: U1.21 (VM), U1.22 (VM), U1.23 (VM), U1.6 (VM), U1.7 (VM), U1.8 (VM)
