File: PCB/IntegratedStepper/Magnetic_Encoder.kicad_sch (KiCad schematic)
At the start: 3 parts, among them U2 AS5048A

Commit message: Update final layout, replace CAN w/ JST
Parts:
- C17: LCSC C2929200 -> C5186689; LCSC Part C2929200 -> C5186689; LCSC Part Number C2929200 -> C5186689
Changed lines of the file:
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@@
 			)
 		)
-		(property "LCSC" "C2929200"
+		(property "LCSC" "C5186689"
 			(at 170.18 80.01 0)
 			(effects
@@
 			)
 		)
-		(property "LCSC Part Number" "C2929200"
+		(property "LCSC Part Number" "C5186689"
 			(at 170.18 80.01 0)
 			(effects
@@
 			)
 		)
-		(property "LCSC Part" "C2929200"
+		(property "LCSC Part" "C5186689"
 			(at 170.18 80.01 0)
 			(effects
