File: PCB/IntegratedStepper/RS485.kicad_sch (KiCad schematic)
At the start: 5 parts, among them IC2 SN65HVD230DR

Commit message: Update final layout, replace CAN w/ JST
Parts:
- C15: LCSC C2929200 -> C5186689; LCSC Part C2929200 -> C5186689; LCSC Part Number C2929200 -> C5186689
- R1: value 10k -> 8.2k; LCSC C469659 -> C25981; LCSC Part C469659 -> C25981; LCSC Part Number C469659 -> C25981
Changed lines of the file:
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@@
 			)
 		)
-		(property "Value" "10k"
+		(property "Value" "8.2k"
 			(at 166.37 99.695 0)
 			(effects
@@
 			)
 		)
-		(property "LCSC" "C469659"
+		(property "LCSC" "C25981"
 			(at 163.83 97.79 0)
 			(effects
@@
 			)
 		)
-		(property "LCSC Part" "C469659"
+		(property "LCSC Part" "C25981"
 			(at 163.83 97.79 0)
 			(effects
@@
 			)
 		)
-		(property "LCSC Part Number" "C469659"
+		(property "LCSC Part Number" "C25981"
 			(at 163.83 97.79 0)
 			(effects
@@
 			)
 		)
-		(property "LCSC" "C2929200"
+		(property "LCSC" "C5186689"
 			(at 194.31 90.17 0)
 			(effects
@@
 			)
 		)
-		(property "LCSC Part Number" "C2929200"
+		(property "LCSC Part Number" "C5186689"
 			(at 194.31 90.17 0)
 			(effects
@@
 			)
 		)
-		(property "LCSC Part" "C2929200"
+		(property "LCSC Part" "C5186689"
 			(at 194.31 90.17 0)
 			(effects
