File: PCB/IntegratedStepper/Stepper_Outputs.kicad_sch (KiCad schematic)
At the start: 6 parts, among them J3 Screw_Terminal_01x02, J4 Screw_Terminal_01x02

Commit message: Update PCB with DRV8243 for 12A capacity
Connections:
- net OUT1: now also J3.2 (Pin_2); no longer J3.1 (Pin_1)
- net OUT2: now also J3.1 (Pin_1); no longer J3.2 (Pin_2)
- net OUT3: now also J4.2 (Pin_2); no longer J4.1 (Pin_1)
- net OUT4: now also J4.1 (Pin_1); no longer J4.2 (Pin_2)
Changed lines of the file:
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@@
 	(symbol
 		(lib_id "Connector:Screw_Terminal_01x02")
-		(at 118.11 59.69 0)
+		(at 118.11 62.23 0)
+		(mirror x)
 		(unit 1)
 		(exclude_from_sim no)
@@
 		(on_board yes)
 		(dnp no)
-		(fields_autoplaced yes)
 		(property "Reference" "J4"
-			(at 120.65 59.6899 0)
+			(at 120.65 62.2301 0)
 			(effects
 				(font
@@
 		)
 		(property "Value" "Screw_Terminal_01x02"
-			(at 120.65 62.2299 0)
+			(at 120.65 59.6901 0)
 			(effects
 				(font
@@
 		)
 		(property "Footprint" "easyeda2kicad:CONN-TH_P5.08_KF128-5.08-2P"
-			(at 118.11 59.69 0)
+			(at 118.11 62.23 0)
 			(effects
 				(font
@@
 		)
 		(property "Datasheet" "~"
-			(at 118.11 59.69 0)
+			(at 118.11 62.23 0)
 			(effects
 				(font
@@
 		)
 		(property "Description" "Generic screw terminal, single row, 01x02, script generated (kicad-library-utils/schlib/autogen/connector/)"
-			(at 118.11 59.69 0)
+			(at 118.11 62.23 0)
 			(effects
 				(font
@@
 		)
 		(property "LCSC" "C474952"
-			(at 118.11 59.69 0)
+			(at 118.11 62.23 0)
 			(effects
 				(font
@@
 		)
 		(property "LCSC Part" "C474952"
-			(at 118.11 59.69 0)
+			(at 118.11 62.23 0)
 			(effects
 				(font
@@
 		)
 		(property "LCSC Part Number" "C474952"
-			(at 118.11 59.69 0)
+			(at 118.11 62.23 0)
 			(effects
 				(font
@@
 	)
 	(symbol
+		(lib_id "Connector:Screw_Terminal_01x02")
+		(at 118.11 55.88 0)
+		(mirror x)
+		(unit 1)
+		(exclude_from_sim no)
+		(in_bom yes)
+		(on_board yes)
+		(dnp no)
+		(property "Reference" "J3"
+			(at 120.65 55.8801 0)
+			(effects
+				(font
+					(size 1.27 1.27)
+				)
+				(justify left)
+			)
+		)
+		(property "Value" "Screw_Terminal_01x02"
+			(at 120.65 53.3401 0)
+			(effects
+				(font
+					(size 1.27 1.27)
+				)
+				(justify left)
+			)
+		)
+		(property "Footprint" "easyeda2kicad:CONN-TH_P5.08_KF128-5.08-2P"
+			(at 118.11 55.88 0)
+			(effects
+				(font
+					(size 1.27 1.27)
+				)
+				(hide yes)
+			)
+		)
+		(property "Datasheet" "~"
+			(at 118.11 55.88 0)
+			(effects
+				(font
+					(size 1.27 1.27)
+				)
+				(hide yes)
+			)
+		)
+		(property "Description" "Generic screw terminal, single row, 01x02, script generated (kicad-library-utils/schlib/autogen/connector/)"
+			(at 118.11 55.88 0)
+			(effects
+				(font
+					(size 1.27 1.27)
+				)
+				(hide yes)
+			)
+		)
+		(property "LCSC" "C474952"
+			(at 118.11 55.88 0)
+			(effects
+				(font
+					(size 1.27 1.27)
+				)
+				(hide yes)
+			)
+		)
+		(property "LCSC Part" "C474952"
+			(at 118.11 55.88 0)
+			(effects
+				(font
+					(size 1.27 1.27)
+				)
+				(hide yes)
+			)
+		)
+		(property "LCSC Part Number" "C474952"
+			(at 118.11 55.88 0)
+			(effects
+				(font
+					(size 1.27 1.27)
+				)
+				(hide yes)
+			)
+		)
+		(pin "2"
+		)
+		(pin "1"
+		)
+		(instances
+			(project "IntegratedStepper"
+				(path "/ab592993-dafc-411a-b466-8e8425f43767/43bbe4fd-5a99-4112-a855-d9b549a4340b"
+					(reference "J3")
+					(unit 1)
+				)
+			)
+		)
+	)
+	(symbol
 		(lib_id "power:GND")
 		(at 158.75 40.64 0)
@@
 					(unit 1)
 				)
-			)
-		)
-	)
-	(symbol
-		(lib_id "Connector:Screw_Terminal_01x02")
-		(at 118.11 53.34 0)
-		(unit 1)
-		(exclude_from_sim no)
-		(in_bom yes)
-		(on_board yes)
-		(dnp no)
-		(fields_autoplaced yes)
-		(property "Reference" "J3"
-			(at 120.65 53.3399 0)
-			(effects
-				(font
-					(size 1.27 1.27)
-				)
-				(justify left)
-			)
-		)
-		(property "Value" "Screw_Terminal_01x02"
-			(at 120.65 55.8799 0)
-			(effects
-				(font
-					(size 1.27 1.27)
-				)
-				(justify left)
-			)
-		)
-		(property "Footprint" "easyeda2kicad:CONN-TH_P5.08_KF128-5.08-2P"
-			(at 118.11 53.34 0)
-			(effects
-				(font
-					(size 1.27 1.27)
-				)
-				(hide yes)
-			)
-		)
-		(property "Datasheet" "~"
-			(at 118.11 53.34 0)
-			(effects
-				(font
-					(size 1.27 1.27)
-				)
-				(hide yes)
-			)
-		)
-		(property "Description" "Generic screw terminal, single row, 01x02, script generated (kicad-library-utils/schlib/autogen/connector/)"
-			(at 118.11 53.34 0)
-			(effects
-				(font
-					(size 1.27 1.27)
-				)
-				(hide yes)
-			)
-		)
-		(property "LCSC" "C474952"
-			(at 118.11 53.34 0)
-			(effects
-				(font
-					(size 1.27 1.27)
-				)
-				(hide yes)
-			)
-		)
-		(property "LCSC Part" "C474952"
-			(at 118.11 53.34 0)
-			(effects
-				(font
-					(size 1.27 1.27)
-				)
-				(hide yes)
-			)
-		)
-		(property "LCSC Part Number" "C474952"
-			(at 118.11 53.34 0)
-			(effects
-				(font
-					(size 1.27 1.27)
-				)
-				(hide yes)
-			)
-		)
-		(pin "2"
-		)
-		(pin "1"
-		)
-		(instances
-			(project "IntegratedStepper"
-				(path "/ab592993-dafc-411a-b466-8e8425f43767/43bbe4fd-5a99-4112-a855-d9b549a4340b"
-					(reference "J3")
-					(unit 1)
-				)

Commit message: update new layout with DRV8245
Connections:
- net OUT1: now also J3.1 (Pin_1); no longer J3.2 (Pin_2)
- net OUT2: now also J3.2 (Pin_2); no longer J3.1 (Pin_1)
- net OUT3: now also J4.1 (Pin_1); no longer J4.2 (Pin_2)
- net OUT4: now also J4.2 (Pin_2); no longer J4.1 (Pin_1)
Other:
- moved on the sheet: J3, J4
Changed lines of the file:
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@@
 	(wire
 		(pts
-			(xy 105.41 53.34) (xy 113.03 53.34)
-		)
-		(stroke
-			(width 0)
-			(type default)
-		)
-	)
-	(wire
-		(pts
-			(xy 105.41 62.23) (xy 113.03 62.23)
+			(xy 105.41 62.23) (xy 114.3 62.23)
 		)
 		(stroke
@@
 	(wire
 		(pts
-			(xy 105.41 55.88) (xy 113.03 55.88)
+			(xy 105.41 53.34) (xy 114.3 53.34)
 		)
 		(stroke
@@
 	(wire
 		(pts
+			(xy 105.41 59.69) (xy 114.3 59.69)
+		)
+		(stroke
+			(width 0)
+			(type default)
+		)
+	)
+	(wire
+		(pts
+			(xy 105.41 55.88) (xy 114.3 55.88)
+		)
+		(stroke
+			(width 0)
+			(type default)
+		)
+	)
+	(wire
+		(pts
 			(xy 147.32 40.64) (xy 154.94 40.64)
 		)
@@
 		(pts
 			(xy 96.52 50.8) (xy 102.87 50.8)
-		)
-		(stroke
-			(width 0)
-			(type default)
-		)
-	)
-	(wire
-		(pts
-			(xy 105.41 59.69) (xy 113.03 59.69)
 		)
 		(stroke
@@
 	(symbol
 		(lib_id "Connector:Screw_Terminal_01x02")
-		(at 118.11 62.23 0)
-		(mirror x)
+		(at 119.38 59.69 0)
 		(unit 1)
 		(exclude_from_sim no)
@@
 		(dnp no)
 		(property "Reference" "J4"
-			(at 120.65 62.2301 0)
+			(at 121.92 59.6899 0)
 			(effects
 				(font
@@
 		)
 		(property "Value" "Screw_Terminal_01x02"
-			(at 120.65 59.6901 0)
+			(at 121.92 62.2299 0)
 			(effects
 				(font
@@
 		)
 		(property "Footprint" "easyeda2kicad:CONN-TH_P5.08_KF128-5.08-2P"
-			(at 118.11 62.23 0)
+			(at 119.38 59.69 0)
 			(effects
 				(font
@@
 		)
 		(property "Datasheet" "~"
-			(at 118.11 62.23 0)
+			(at 119.38 59.69 0)
 			(effects
 				(font
@@
 		)
 		(property "Description" "Generic screw terminal, single row, 01x02, script generated (kicad-library-utils/schlib/autogen/connector/)"
-			(at 118.11 62.23 0)
+			(at 119.38 59.69 0)
 			(effects
 				(font
@@
 		)
 		(property "LCSC" "C474952"
-			(at 118.11 62.23 0)
+			(at 119.38 59.69 0)
 			(effects
 				(font
@@
 		)
 		(property "LCSC Part" "C474952"
-			(at 118.11 62.23 0)
+			(at 119.38 59.69 0)
 			(effects
 				(font
@@
 		)
 		(property "LCSC Part Number" "C474952"
-			(at 118.11 62.23 0)
+			(at 119.38 59.69 0)
 			(effects
 				(font
@@
 	(symbol
 		(lib_id "Connector:Screw_Terminal_01x02")
-		(at 118.11 55.88 0)
-		(mirror x)
+		(at 119.38 53.34 0)
 		(unit 1)
 		(exclude_from_sim no)
@@
 		(dnp no)
 		(property "Reference" "J3"
-			(at 120.65 55.8801 0)
+			(at 121.92 53.3399 0)
 			(effects
 				(font
@@
 		)
 		(property "Value" "Screw_Terminal_01x02"
-			(at 120.65 53.3401 0)
+			(at 121.92 55.8799 0)
 			(effects
 				(font
@@
 		)
 		(property "Footprint" "easyeda2kicad:CONN-TH_P5.08_KF128-5.08-2P"
-			(at 118.11 55.88 0)
+			(at 119.38 53.34 0)
 			(effects
 				(font
@@
 		)
 		(property "Datasheet" "~"
-			(at 118.11 55.88 0)
+			(at 119.38 53.34 0)
 			(effects
 				(font
@@
 		)
 		(property "Description" "Generic screw terminal, single row, 01x02, script generated (kicad-library-utils/schlib/autogen/connector/)"
-			(at 118.11 55.88 0)
+			(at 119.38 53.34 0)
 			(effects
 				(font
@@
 		)
 		(property "LCSC" "C474952"
-			(at 118.11 55.88 0)
+			(at 119.38 53.34 0)
 			(effects
 				(font
@@
 		)
 		(property "LCSC Part" "C474952"
-			(at 118.11 55.88 0)
+			(at 119.38 53.34 0)
 			(effects
 				(font
@@
 		)
 		(property "LCSC Part Number" "C474952"
-			(at 118.11 55.88 0)
-			(effects
-				(font
+			(at 119.38 53.34 0)
+			(effects
+				(font
